File: ice40HX1K-SRAM/power.sch (KiCad schematic (older format))
At the start: 22 parts, among them J1 Conn_01x03_Male, U1 LTC3406ES5, U2 MAX40200AUK, U3 LTC3406ES5, U4 MAX40200AUK

Commit message: starting layout
Parts:
- BT1: footprint (none) -> kifootp:CR2032
- C57: footprint (none) -> Capacitor_SMD:C_0402_1005Metric
- L1, L2: footprint Inductor_SMD:L_1210_3225Metric -> Inductor_SMD:L_0805_2012Metric
Changed lines of the file:
@@
 F 0 "L1" V 2519 2400 50  0000 C CNN
 F 1 "2.2uH" V 2610 2400 50  0000 C CNN
-F 2 "Inductor_SMD:L_1210_3225Metric" H 2700 2400 50  0001 C CNN
+F 2 "Inductor_SMD:L_0805_2012Metric" H 2700 2400 50  0001 C CNN
 F 3 "~" H 2700 2400 50  0001 C CNN
 	1    2700 2400
@@
 F 0 "L2" V 5469 2450 50  0000 C CNN
 F 1 "2.2uH" V 5560 2450 50  0000 C CNN
-F 2 "Inductor_SMD:L_1210_3225Metric" H 5650 2450 50  0001 C CNN
+F 2 "Inductor_SMD:L_0805_2012Metric" H 5650 2450 50  0001 C CNN
 F 3 "~" H 5650 2450 50  0001 C CNN
 	1    5650 2450
@@
 F 0 "BT1" H 3068 5046 50  0000 L CNN
 F 1 "Battery_Cell" H 3068 4955 50  0000 L CNN
-F 2 "" V 2950 5010 50  0001 C CNN
+F 2 "kifootp:CR2032" V 2950 5010 50  0001 C CNN
 F 3 "~" V 2950 5010 50  0001 C CNN
 	1    2950 4950
@@
 F 0 "C57" H 3515 5046 50  0000 L CNN
 F 1 "0.1uF" H 3515 4955 50  0000 L CNN
-F 2 "" H 3438 4850 50  0001 C CNN
+F 2 "Capacitor_SMD:C_0402_1005Metric" H 3438 4850 50  0001 C CNN
 F 3 "~" H 3400 5000 50  0001 C CNN
 	1    3400 5000
