File: ice40HX1K-SRAM/HX1KADCboard.kicad_pcb (KiCad board)
At the start: 2 copper layers, 124.5 x 96.5 mm, 45 parts, among them J1 Conn_02x05_Odd_Even, J2 Conn_01x20_Male, J5 Conn_01x20_Male, J6 Conn_01x03_Male, U1 LTC3406ES5, U2 AT25SF081-SSHD-X, U3 ICE40HX1K-VQ100(VQFP100), U4 AS7C34096A

Commit message: wiring FPGA
Parts:
- removed C1: 4.7uF, Capacitor_SMD:C_1206_3216Metric
- removed C10, C11, C12, C13, C14, C15, C16, C17, C18, C19, C2, C4, C5, C6, C7, C8, C9: 0.1uF, Capacitor_SMD:C_0805_2012Metric
- removed C3: 10uF, Capacitor_SMD:C_1206_3216Metric
- removed D1: D, Capacitor_SMD:C_0603_1608Metric
- removed D2, D3, D4, D5: LED, LED_SMD:LED_1206_3216Metric
- removed J1: Conn_02x05_Odd_Even, Connector_PinHeader_2.54mm:PinHeader_2x05_P2.54mm_Vertical
- removed J2, J5: Conn_01x20_Male, Connector_PinHeader_2.54mm:PinHeader_1x20_P2.54mm_Vertical
- removed J6: Conn_01x03_Male, Connector_PinHeader_2.54mm:PinHeader_1x03_P2.54mm_Vertical
- removed L1: 2.2uH, Inductor_SMD:L_1210_3225Metric
- removed R1, R2, R3, R4, R5, R6: R, Resistor_SMD:R_1206_3216Metric
- removed R10, R11, R12, R9: 10kohm, Resistor_SMD:R_1206_3216Metric
- removed R7, R8: 100kOhm, Resistor_SMD:R_1206_3216Metric
- removed U1: LTC3406ES5, Package_TO_SOT_SMD:TSOT-23-5
- removed U2: AT25SF081-SSHD-X, Package_SO:SOIC-8_3.9x4.9mm_P1.27mm
- removed U3: ICE40HX1K-VQ100(VQFP100), Package_QFP:LQFP-100_14x14mm_P0.5mm
- removed U4: AS7C34096A, Package_SO:TSOP-II-44_10.16x18.41mm_P0.8mm
Routing:
- net +3V3: track 441.6 -> 0.00 mm, vias 2 -> 0
- net +1V2: track 185.3 -> 0.00 mm, vias 5 -> 0
- net IO1: track 88.9 -> 0.00 mm
- net IO2: track 87.4 -> 0.00 mm
- net CDONE: track 75.6 -> 0.00 mm, vias 3 -> 0
- net IO3: track 70.4 -> 0.00 mm
- net IO4: track 67.7 -> 0.00 mm
- net CRESET: track 66.5 -> 0.00 mm, vias 3 -> 0
- net IO7: track 61.3 -> 0.00 mm
- net IO8: track 59.7 -> 0.00 mm
- net IO9: track 58.8 -> 0.00 mm
- net SPI_SCK: track 58.6 -> 0.00 mm, vias 4 -> 0
- net IO10: track 58.6 -> 0.00 mm
- net SPI_CS: track 57.0 -> 0.00 mm
- net IO43: track 54.6 -> 0.00 mm
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Other:
- board outline removed

Commit message: starting layout
Parts:
- added BT1: Battery_Cell, kifootp:CR2032, F.Cu at (185.2, 53.1)
- added C1: 4.7uF, Capacitor_SMD:C_0402_1005Metric, F.Cu at (194.3, 63.5)
- added C10: 0.1uF, Capacitor_SMD:C_0402_1005Metric, F.Cu at (177.4, 126.6)
- added C11: 0.1uF, Capacitor_SMD:C_0402_1005Metric, F.Cu at (141.8, 60.4)
- added C12: 0.1uF, Capacitor_SMD:C_0402_1005Metric, F.Cu at (145.8, 55.9)
- added C13: 0.1uF, Capacitor_SMD:C_0402_1005Metric, F.Cu at (144.7, 58.4)
- added C14: 0.1uF, Capacitor_SMD:C_0402_1005Metric, F.Cu at (141.8, 66.4)
- added C15: 0.1uF, Capacitor_SMD:C_0402_1005Metric, F.Cu at (141.8, 58.4)
- added C16: 0.1uF, Capacitor_SMD:C_0402_1005Metric, F.Cu at (150.5, 57.9)
- added C17: 0.1uF, Capacitor_SMD:C_0402_1005Metric, F.Cu at (144.7, 62.4)
- added C18: 0.1uF, Capacitor_SMD:C_0402_1005Metric, F.Cu at (147.6, 59.9)
- added C19: 0.1uF, Capacitor_SMD:C_0402_1005Metric, F.Cu at (151.6, 55.9)
- added C2: 10uF, Capacitor_SMD:C_0603_1608Metric, F.Cu at (205.8, 54.0)
- added C20: 0.1uF, Capacitor_SMD:C_0402_1005Metric, F.Cu at (141.8, 64.4)
- added C21: 0.1uF, Capacitor_SMD:C_0402_1005Metric, F.Cu at (147.6, 57.9)
- added C22: 0.1uF, Capacitor_SMD:C_0402_1005Metric, F.Cu at (144.7, 60.4)
- added C23: 0.1uF, Capacitor_SMD:C_0402_1005Metric, F.Cu at (141.8, 62.4)
- added C24: 0.1uF, Capacitor_SMD:C_0402_1005Metric, F.Cu at (148.7, 55.9)
- added C25: 0.1uF, Capacitor_SMD:C_0402_1005Metric, F.Cu at (99.0, 84.9)
- added C26: 0.1uF, Capacitor_SMD:C_0402_1005Metric, F.Cu at (96.0, 84.9)
- added C27: 4.7uF, Capacitor_SMD:C_0402_1005Metric, F.Cu at (134.9, 138.9)
- added C28: 0.1uF, Capacitor_SMD:C_0402_1005Metric, F.Cu at (153.9, 124.6)
- added C29: 4.7uF, Capacitor_SMD:C_0402_1005Metric, F.Cu at (188.2, 114.3)
- added C3: 4.7uF, Capacitor_SMD:C_0402_1005Metric, F.Cu at (197.2, 63.5)
- added C30: 0.1uF, Capacitor_SMD:C_0402_1005Metric, F.Cu at (178.9, 113.8)
- added C31: 0.01uF, Capacitor_SMD:C_0402_1005Metric, F.Cu at (219.7, 82.5)
- added C32: 0.01uF, Capacitor_SMD:C_0402_1005Metric, F.Cu at (228.3, 74.9)
- added C33: 0.01uF, Capacitor_SMD:C_0402_1005Metric, F.Cu at (233.4, 70.4)
- added C34: 0.01uF, Capacitor_SMD:C_0402_1005Metric, F.Cu at (222.6, 82.5)
- added C35: 0.01uF, Capacitor_SMD:C_0402_1005Metric, F.Cu at (233.4, 72.4)
- added C36: 0.01uF, Capacitor_SMD:C_0402_1005Metric, F.Cu at (231.2, 74.9)
- added C37: 100pF, Capacitor_SMD:C_0402_1005Metric, F.Cu at (104.5, 50.3)
- added C38: 100pF, Capacitor_SMD:C_0402_1005Metric, F.Cu at (104.5, 52.3)
- added C39: Ccap, kifootp:CAPBUTTON, F.Cu at (64.8, 51.8)
- added C4: 0.1uF, Capacitor_SMD:C_0402_1005Metric, F.Cu at (209.3, 49.1)
- added C40: Ccap, kifootp:CAPBUTTON, F.Cu at (64.8, 64.8)
- added C41: 100pF, Capacitor_SMD:C_0402_1005Metric, F.Cu at (104.5, 48.3)
- added C42: 100pF, Capacitor_SMD:C_0402_1005Metric, F.Cu at (101.6, 52.3)
- added C43: Ccap, kifootp:CAPBUTTON, F.Cu at (77.8, 51.8)
- added C44: Ccap, kifootp:CAPBUTTON, F.Cu at (90.7, 64.8)
- added C45: 100pF, Capacitor_SMD:C_0402_1005Metric, F.Cu at (101.6, 50.3)
- added C46: 100pF, Capacitor_SMD:C_0402_1005Metric, F.Cu at (98.7, 46.3)
- added C47: Ccap, kifootp:CAPBUTTON, F.Cu at (90.7, 51.8)
- added C48: Ccap, kifootp:CAPBUTTON, F.Cu at (77.8, 64.8)
- added C49: 10uF, Capacitor_SMD:C_0603_1608Metric, F.Cu at (174.0, 87.6)
- added C5: 10uF, Capacitor_SMD:C_0603_1608Metric, F.Cu at (186.8, 63.7)
- added C50: 10uF, Capacitor_SMD:C_0603_1608Metric, F.Cu at (178.0, 87.6)
- added C51: 1uF, Capacitor_SMD:C_0402_1005Metric, F.Cu at (200.1, 80.5)
- added C52: 1uF, Capacitor_SMD:C_0402_1005Metric, F.Cu at (195.9, 83.9)
- added C53: 10uF, Capacitor_SMD:C_0603_1608Metric, F.Cu at (182.0, 87.6)
- added C54: 10uF, Capacitor_SMD:C_0603_1608Metric, F.Cu at (186.0, 87.6)
- added C55: 1uF, Capacitor_SMD:C_0402_1005Metric, F.Cu at (193.3, 85.9)
- added C56: 1uF, Capacitor_SMD:C_0402_1005Metric, F.Cu at (203.1, 76.3)
- added C57: 0.1uF, Capacitor_SMD:C_0402_1005Metric, F.Cu at (209.3, 51.1)
- added C6: 10uF, Capacitor_SMD:C_0603_1608Metric, F.Cu at (182.8, 63.7)
- added C7: 0.1uF, Capacitor_SMD:C_0402_1005Metric, F.Cu at (209.9, 44.7)
- added C8: 0.1uF, Capacitor_SMD:C_0402_1005Metric, F.Cu at (209.9, 46.7)
- added C9: 10uF, Capacitor_SMD:C_0603_1608Metric, F.Cu at (190.8, 63.7)
- added D1: LED, LED_SMD:LED_1206_3216Metric, F.Cu at (156.4, 90.7)
- added D10: LED, LED_SMD:LED_1206_3216Metric, F.Cu at (189.6, 101.5)
- added D11: LED, LED_SMD:LED_1206_3216Metric, F.Cu at (197.4, 71.1)
- added D12: LED, LED_SMD:LED_1206_3216Metric, F.Cu at (180.5, 84.7)
- added D13: LED, LED_SMD:LED_1206_3216Metric, F.Cu at (191.8, 74.5)
- added D14: LED, LED_SMD:LED_1206_3216Metric, F.Cu at (186.1, 84.7)
- added D15: LED, LED_SMD:LED_1206_3216Metric, F.Cu at (197.4, 74.5)
- added D16: LED, LED_SMD:LED_1206_3216Metric, F.Cu at (191.8, 77.9)
- added D17: LED, LED_SMD:LED_1206_3216Metric, F.Cu at (186.1, 81.3)
- added D18: LED, LED_SMD:LED_1206_3216Metric, F.Cu at (174.8, 74.5)
- added D19: LED, LED_SMD:LED_1206_3216Metric, F.Cu at (180.5, 71.1)
- added D2: LED, LED_SMD:LED_1206_3216Metric, F.Cu at (156.4, 85.0)
- added D20: LED, LED_SMD:LED_1206_3216Metric, F.Cu at (174.8, 77.9)
- added D21: LED, LED_SMD:LED_1206_3216Metric, F.Cu at (180.5, 74.5)
- added D22: LED, LED_SMD:LED_1206_3216Metric, F.Cu at (174.8, 71.1)
- added D23: LED, LED_SMD:LED_1206_3216Metric, F.Cu at (186.1, 71.1)
- added D24: LED, LED_SMD:LED_1206_3216Metric, F.Cu at (174.8, 81.3)
- added D25: LED, LED_SMD:LED_1206_3216Metric, F.Cu at (180.5, 77.9)
- added D26: LED, LED_SMD:LED_1206_3216Metric, F.Cu at (186.1, 74.5)
- added D27: LED, LED_SMD:LED_1206_3216Metric, F.Cu at (174.8, 84.7)
- added D28: LED, LED_SMD:LED_1206_3216Metric, F.Cu at (191.8, 71.1)
- added D29: LED, LED_SMD:LED_1206_3216Metric, F.Cu at (180.5, 81.3)
- added D3: LED, LED_SMD:LED_1206_3216Metric, F.Cu at (156.4, 79.4)
- added D30: LED, LED_SMD:LED_1206_3216Metric, F.Cu at (186.1, 77.9)
- added D4: LED, LED_SMD:LED_1206_3216Metric, F.Cu at (156.4, 96.3)
- added D5: CDBU05, Capacitor_SMD:C_0603_1608Metric, F.Cu at (142.3, 56.2)
- added D6: LED, LED_SMD:LED_1206_3216Metric, F.Cu at (146.2, 132.3)
- added D7: LED, LED_SMD:LED_1206_3216Metric, F.Cu at (189.6, 111.6)
- added D8: LED, LED_SMD:LED_1206_3216Metric, F.Cu at (189.6, 108.2)
- added D9: LED, LED_SMD:LED_1206_3216Metric, F.Cu at (189.6, 104.9)
- added J1: Conn_01x03_Male, Connector_PinHeader_2.54mm:PinHeader_1x03_P2.54mm_Vertical, F.Cu at (200.7, 46.0)
- added J2: Conn_02x05_Odd_Even, Connector_PinHeader_2.54mm:PinHeader_2x05_P2.54mm_Vertical, F.Cu at (168.1, 121.4)
- added J3: Conn_01x20_Male, Connector_PinHeader_2.54mm:PinHeader_1x20_P2.54mm_Vertical, F.Cu at (111.3, 42.6)
- added J5: Conn_01x06_Male, Connector_PinHeader_2.54mm:PinHeader_1x06_P2.54mm_Vertical, F.Cu at (128.2, 125.9)
- added J6: Conn_01x05, Connector_PinHeader_2.54mm:PinHeader_1x05_P2.54mm_Vertical, F.Cu at (184.4, 102.1)
- added L1: 2.2uH, Inductor_SMD:L_0805_2012Metric, F.Cu at (178.6, 64.0)
- added L2: 2.2uH, Inductor_SMD:L_0805_2012Metric, F.Cu at (174.2, 64.0)
- added L3: 10uH, Inductor_SMD:L_0805_2012Metric, F.Cu at (196.8, 77.7)
- added L4: 10uH, Inductor_SMD:L_0805_2012Metric, F.Cu at (191.1, 81.1)
- added L5: 10uH, Inductor_SMD:L_0805_2012Metric, F.Cu at (202.4, 70.9)
- added L6: 10uH, Inductor_SMD:L_0805_2012Metric, F.Cu at (202.4, 73.8)
- added R1: 100kOhm, Resistor_SMD:R_0402_1005Metric, F.Cu at (205.2, 56.3)
- added R10: 10kOhm, Resistor_SMD:R_0402_1005Metric, F.Cu at (182.9, 122.1)
- added R11: 10kohm, Resistor_SMD:R_0402_1005Metric, F.Cu at (155.7, 66.4)
- added R12: 10kohm, Resistor_SMD:R_0402_1005Metric, F.Cu at (155.7, 69.3)
- added R13: 10kohm, Resistor_SMD:R_0402_1005Metric, F.Cu at (155.7, 72.2)
- added R14: 10kohm, Resistor_SMD:R_0402_1005Metric, F.Cu at (155.7, 75.1)
- added R15: 10kOhm, Resistor_SMD:R_0402_1005Metric, F.Cu at (131.9, 138.9)
- added R16: 10kOhm, Resistor_SMD:R_0402_1005Metric, F.Cu at (176.0, 113.8)
- added R17: 10kOhm, Resistor_SMD:R_0402_1005Metric, F.Cu at (173.1, 113.8)
- added R18: 10kOhm, Resistor_SMD:R_0402_1005Metric, F.Cu at (170.2, 113.8)
- added R19: 10kOhm, Resistor_SMD:R_0402_1005Metric, F.Cu at (167.3, 113.8)
- added R2: 100kOhm, Resistor_SMD:R_0402_1005Metric, F.Cu at (204.7, 58.8)
- added R20: 100kOhm, Resistor_SMD:R_0402_1005Metric, F.Cu at (98.7, 52.3)
- added R21: 100kOhm, Resistor_SMD:R_0402_1005Metric, F.Cu at (98.7, 50.3)
- added R22: 100kOhm, Resistor_SMD:R_0402_1005Metric, F.Cu at (101.6, 48.3)
- added R23: 100kOhm, Resistor_SMD:R_0402_1005Metric, F.Cu at (98.7, 48.3)
- added R24: 100kOhm, Resistor_SMD:R_0402_1005Metric, F.Cu at (104.5, 46.3)
- added R25: 100kOhm, Resistor_SMD:R_0402_1005Metric, F.Cu at (101.6, 46.3)
- added R26: 20Ohm, Resistor_SMD:R_0402_1005Metric, F.Cu at (190.4, 86.8)
- added R27: 20Ohm, Resistor_SMD:R_0402_1005Metric, F.Cu at (203.1, 78.3)
- added R28: 20Ohm, Resistor_SMD:R_0402_1005Metric, F.Cu at (193.0, 83.9)
- added R29: 20Ohm, Resistor_SMD:R_0402_1005Metric, F.Cu at (200.1, 82.5)
- added R3: 100kOhm, Resistor_SMD:R_0402_1005Metric, F.Cu at (200.1, 63.5)
- added R4: 450kOhm, Resistor_SMD:R_0402_1005Metric, F.Cu at (209.2, 53.8)
- added R5: 10kOhm, Resistor_SMD:R_0402_1005Metric, F.Cu at (174.5, 128.6)
- added R6: 10kOhm, Resistor_SMD:R_0402_1005Metric, F.Cu at (174.5, 126.6)
- added R7: 10kOhm, Resistor_SMD:R_0402_1005Metric, F.Cu at (182.9, 120.1)
- added R8: 10kOhm, Resistor_SMD:R_0402_1005Metric, F.Cu at (185.8, 120.1)
- added R9: 10kOhm, Resistor_SMD:R_0402_1005Metric, F.Cu at (174.5, 130.5)
- added U1: LTC3406ES5, Package_TO_SOT_SMD:TSOT-23-5, F.Cu at (201.1, 55.6)
- added U10: FAN5341, kifootp:FAN5341, F.Cu at (190.2, 84.2)
- added U11: FAN5341, kifootp:FAN5341, F.Cu at (197.3, 80.8)
- added U12: FAN5341, kifootp:FAN5341, F.Cu at (194.7, 81.2)
- added U13: FAN5341, kifootp:FAN5341, F.Cu at (200.3, 77.8)
- added U2: MAX40200AUK, Package_TO_SOT_SMD:SOT-23-5, F.Cu at (200.8, 60.2)
- added U3: LTC3406ES5, Package_TO_SOT_SMD:TSOT-23-5, F.Cu at (205.7, 45.9)
- added U4: MAX40200AUK, Package_TO_SOT_SMD:SOT-23-5, F.Cu at (205.4, 50.5)
- added U5: AT25SF081-SSHD-X, Package_SO:SOIC-8_3.9x4.9mm_P1.27mm, F.Cu at (177.2, 122.3)
- added U6: ICE40HX1K-VQ100(VQFP100), Package_QFP:LQFP-100_14x14mm_P0.5mm, F.Cu at (131.1, 64.2)
- added U7: AS7C34096A, Package_SO:TSOP-II-44_10.16x18.41mm_P0.8mm, F.Cu at (107.5, 75.9)
- added U8: ATSAMD11D14A-SS, Package_SO:SOIC-20W_7.5x12.8mm_P1.27mm, F.Cu at (136.9, 130.8)
- added U9: BL652, RF_Module:Laird_BL652, F.Cu at (174.6, 106.3)
- added X1: USBFCI_10103594_MILL, kifootp:FCI_10103594_MILL, F.Cu at (147.9, 129.8)
- added X2: ASE-10MHz, Oscillator:Oscillator_SMD_Abracon_ASE-4Pin_3.2x2.5mm, F.Cu at (225.8, 79.3)
- added X3: ASE-10MHz, Oscillator:Oscillator_SMD_Abracon_ASE-4Pin_3.2x2.5mm, F.Cu at (229.4, 71.6)
- added X4: ASE-10MHz, Oscillator:Oscillator_SMD_Abracon_ASE-4Pin_3.2x2.5mm, F.Cu at (220.7, 79.3)
- added X5: ASV-xxxMHz, Oscillator:Oscillator_SMD_Abracon_ASV-4Pin_7.0x5.1mm, F.Cu at (213.9, 80.9)
- added X6: ASV-xxxMHz, Oscillator:Oscillator_SMD_Abracon_ASV-4Pin_7.0x5.1mm, F.Cu at (213.9, 73.2)
- added X7: ASV-xxxMHz, Oscillator:Oscillator_SMD_Abracon_ASV-4Pin_7.0x5.1mm, F.Cu at (222.5, 73.2)

Commit message: starting layout
Parts:
- moved C11 31.3 mm to (110.5, 58.8)
- moved C12 31.3 mm to (114.5, 54.3)
- moved C14 31.3 mm to (110.5, 64.7)
- moved C16 31.3 mm to (119.2, 56.2)
- moved C13 19.7 mm to (135.3, 75.7)
- moved C15 19.7 mm to (132.4, 75.7)
- moved C17 19.7 mm to (135.3, 79.7)
- moved C18 19.7 mm to (138.2, 77.2)
- moved C21 16.7 mm to (133.5, 49.0)
- moved C23 16.7 mm to (127.7, 53.5)
- moved C19 16.7 mm to (137.5, 47.1)
- moved C24 3.63 mm to (148.6, 59.5)
- moved C20 3.63 mm to (141.7, 68.0)
- moved C22 3.63 mm to (144.6, 64.0)
Changed lines of the file:
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@@
   )
   (module Capacitor_SMD:C_0402_1005Metric (layer F.Cu)
-    (at 148.701001 55.911001)
+    (at 148.591001 59.541001)
     (descr "Capacitor SMD 0402 (1005 Metric), square (rectangular) end terminal, IPC_7351 nominal, (Body size source: http://www.tortai-tech.com/upload/download/2011102023233369053.pdf), generated with kicad-footprint-generator")
     (tags capacitor)
@@
   )
   (module Capacitor_SMD:C_0402_1005Metric (layer F.Cu)
-    (at 141.781001 62.401001)
+    (at 127.661001 53.541001)
     (descr "Capacitor SMD 0402 (1005 Metric), square (rectangular) end terminal, IPC_7351 nominal, (Body size source: http://www.tortai-tech.com/upload/download/2011102023233369053.pdf), generated with kicad-footprint-generator")
     (tags capacitor)
@@
   )
   (module Capacitor_SMD:C_0402_1005Metric (layer F.Cu)
-    (at 144.691001 60.411001)
+    (at 144.581001 64.041001)
     (descr "Capacitor SMD 0402 (1005 Metric), square (rectangular) end terminal, IPC_7351 nominal, (Body size source: http://www.tortai-tech.com/upload/download/2011102023233369053.pdf), generated with kicad-footprint-generator")
     (tags capacitor)
@@
   )
   (module Capacitor_SMD:C_0402_1005Metric (layer F.Cu)
-    (at 147.601001 57.901001)
+    (at 133.481001 49.041001)
     (descr "Capacitor SMD 0402 (1005 Metric), square (rectangular) end terminal, IPC_7351 nominal, (Body size source: http://www.tortai-tech.com/upload/download/2011102023233369053.pdf), generated with kicad-footprint-generator")
     (tags capacitor)
@@
   )
   (module Capacitor_SMD:C_0402_1005Metric (layer F.Cu)
-    (at 141.781001 64.391001)
+    (at 141.671001 68.021001)
     (descr "Capacitor SMD 0402 (1005 Metric), square (rectangular) end terminal, IPC_7351 nominal, (Body size source: http://www.tortai-tech.com/upload/download/2011102023233369053.pdf), generated with kicad-footprint-generator")
     (tags capacitor)
@@
   )
   (module Capacitor_SMD:C_0402_1005Metric (layer F.Cu)
-    (at 151.611001 55.911001)
+    (at 137.491001 47.051001)
     (descr "Capacitor SMD 0402 (1005 Metric), square (rectangular) end terminal, IPC_7351 nominal, (Body size source: http://www.tortai-tech.com/upload/download/2011102023233369053.pdf), generated with kicad-footprint-generator")
     (tags capacitor)
@@
   )
   (module Capacitor_SMD:C_0402_1005Metric (layer F.Cu)
-    (at 147.601001 59.891001)
+    (at 138.191001 77.161001)
     (descr "Capacitor SMD 0402 (1005 Metric), square (rectangular) end terminal, IPC_7351 nominal, (Body size source: http://www.tortai-tech.com/upload/download/2011102023233369053.pdf), generated with kicad-footprint-generator")
     (tags capacitor)
@@
   )
   (module Capacitor_SMD:C_0402_1005Metric (layer F.Cu)
-    (at 144.691001 62.401001)
+    (at 135.281001 79.671001)
     (descr "Capacitor SMD 0402 (1005 Metric), square (rectangular) end terminal, IPC_7351 nominal, (Body size source: http://www.tortai-tech.com/upload/download/2011102023233369053.pdf), generated with kicad-footprint-generator")
     (tags capacitor)
@@
   )
   (module Capacitor_SMD:C_0402_1005Metric (layer F.Cu)
-    (at 150.511001 57.901001)
+    (at 119.211001 56.241001)
     (descr "Capacitor SMD 0402 (1005 Metric), square (rectangular) end terminal, IPC_7351 nominal, (Body size source: http://www.tortai-tech.com/upload/download/2011102023233369053.pdf), generated with kicad-footprint-generator")
     (tags capacitor)
@@
   )
   (module Capacitor_SMD:C_0402_1005Metric (layer F.Cu)
-    (at 141.781001 58.421001)
+    (at 132.371001 75.691001)
     (descr "Capacitor SMD 0402 (1005 Metric), square (rectangular) end terminal, IPC_7351 nominal, (Body size source: http://www.tortai-tech.com/upload/download/2011102023233369053.pdf), generated with kicad-footprint-generator")
     (tags capacitor)
@@
   )
   (module Capacitor_SMD:C_0402_1005Metric (layer F.Cu)
-    (at 141.781001 66.381001)
+    (at 110.481001 64.721001)
     (descr "Capacitor SMD 0402 (1005 Metric), square (rectangular) end terminal, IPC_7351 nominal, (Body size source: http://www.tortai-tech.com/upload/download/2011102023233369053.pdf), generated with kicad-footprint-generator")
     (tags capacitor)
@@
   )
   (module Capacitor_SMD:C_0402_1005Metric (layer F.Cu)
-    (at 144.691001 58.421001)
+    (at 135.281001 75.691001)
     (descr "Capacitor SMD 0402 (1005 Metric), square (rectangular) end terminal, IPC_7351 nominal, (Body size source: http://www.tortai-tech.com/upload/download/2011102023233369053.pdf), generated with kicad-footprint-generator")
     (tags capacitor)
@@
   )
   (module Capacitor_SMD:C_0402_1005Metric (layer F.Cu)
-    (at 145.791001 55.911001)
+    (at 114.491001 54.251001)
     (descr "Capacitor SMD 0402 (1005 Metric), square (rectangular) end terminal, IPC_7351 nominal, (Body size source: http://www.tortai-tech.com/upload/download/2011102023233369053.pdf), generated with kicad-footprint-generator")
     (tags capacitor)
@@
   )
   (module Capacitor_SMD:C_0402_1005Metric (layer F.Cu)
-    (at 141.781001 60.411001)
-    (descr "Capacitor SMD 0402 (1005 Metric), square (rectangular) end terminal, IPC_7351 nominal, (Body size source: http://www.tortai-tech.com/upload/download/2011102023233369053.pdf), generated with kicad-footprint-generator")
-    (tags capacitor)
+    (at 110.481001 58.751001)
+    (descr "Capacitor SMD 0402 (1005 Metric), square (rectangular) end terminal, IPC_7351 nominal, (Body size source: http://www.tortai-tech.com/upload/download/2011102023233369053.pdf), generated with kicad-footprint-generator")
+    (tags capacitor)

Commit message: starting AutoRoute
Parts:
- moved C8 130.0 mm to (97.1, 111.4), turned to 270 degrees
- moved C4 119.6 mm to (107.1, 111.2), turned to 270 degrees
- moved BT1 112.7 mm to (84.9, 104.6)
- moved U2 112.7 mm to (100.5, 111.7)
- moved C9 98.5 mm to (104.8, 111.8), turned to 270 degrees
- moved U3 97.2 mm to (143.6, 120.7)
- moved C7 95.2 mm to (153.6, 121.5), turned to 270 degrees
- moved R4 93.4 mm to (141.1, 117.8), turned to 180 degrees
- moved U4 86.6 mm to (156.5, 121.9)
- moved C57 84.0 mm to (163.1, 121.3), turned to 270 degrees
- moved X3 80.7 mm to (151.1, 52.0), turned to 90 degrees
- moved C36 80.4 mm to (154.3, 51.5), turned to 90 degrees
- moved C3 79.8 mm to (144.4, 123.4), turned to 180 degrees
- moved R3 77.3 mm to (145.1, 117.8)
- moved C6 74.8 mm to (141.1, 125.8)
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Routing:
- added copper zone on In2.Cu, net +3V3
- added copper zone on In1.Cu, net GND
Other:
- board outline added: 141.9 x 92.2 mm
- copper layers 2 -> 4

Commit message: starting AutoRoute - fail
Routing:
- net +3V3: track 0.00 -> 141.4 mm, vias 0 -> 58
- net Net-(BT1-Pad1): track 0.00 -> 109.5 mm
- net CDONE: track 0.00 -> 102.2 mm, vias 0 -> 6
- net +1V2: track 0.00 -> 98.1 mm, vias 0 -> 3
- net SPI_SCK: track 0.00 -> 87.3 mm, vias 0 -> 4
- net SPI_OUT: track 0.00 -> 86.7 mm, vias 0 -> 3
- net CRESET: track 0.00 -> 85.3 mm, vias 0 -> 6
- net IO97: track 0.00 -> 83.8 mm, vias 0 -> 2
- net SPI_CS: track 0.00 -> 80.8 mm, vias 0 -> 3
- net SPI_IN: track 0.00 -> 78.0 mm, vias 0 -> 3
- net IO96: track 0.00 -> 75.6 mm, vias 0 -> 2
- net IO95: track 0.00 -> 71.2 mm, vias 0 -> 3
- net IO94: track 0.00 -> 64.0 mm, vias 0 -> 2
- net IO74: track 0.00 -> 57.0 mm
- net IO64: track 0.00 -> 56.3 mm, vias 0 -> 2
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
Commit message: starting AutoRoute - fail
Routing:
- net GND: track 13.2 -> 16.8 mm, vias 290 -> 289
- net +3V3: track 141.4 -> 142.8 mm
Changed lines of the file:
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@@
     (thickness 1.6)
     (drawings 4)
-    (tracks 1661)
+    (tracks 1668)
     (zones 0)
     (modules 148)
@@
   (via (at 133.87 116.04) (size 0.5) (drill 0.25) (layers F.Cu B.Cu) (net 1))
   (via (at 130.22 116.06) (size 0.5) (drill 0.25) (layers F.Cu B.Cu) (net 1))
-  (via (at 126.79 115.38) (size 0.5) (drill 0.25) (layers F.Cu B.Cu) (net 1))
+  (via (at 126.57 115.36) (size 0.5) (drill 0.25) (layers F.Cu B.Cu) (net 1))
   (via (at 124.7 116.25) (size 0.5) (drill 0.25) (layers F.Cu B.Cu) (net 1))
   (via (at 122.48 116.27) (size 0.5) (drill 0.25) (layers F.Cu B.Cu) (net 1))
@@
   (via (at 163.18 117.84) (size 0.5) (drill 0.25) (layers F.Cu B.Cu) (net 1))
   (via (at 161.09 117.31) (size 0.5) (drill 0.25) (layers F.Cu B.Cu) (net 1))
-  (via (at 140.57 111.46) (size 0.5) (drill 0.25) (layers F.Cu B.Cu) (net 1))
+  (via (at 140.49 110.98) (size 0.5) (drill 0.25) (layers F.Cu B.Cu) (net 1))
   (via (at 147.93 116.53) (size 0.5) (drill 0.25) (layers F.Cu B.Cu) (net 1))
   (via (at 144.18 114.88) (size 0.5) (drill 0.25) (layers F.Cu B.Cu) (net 1))
-  (via (at 138.79 113.7) (size 0.5) (drill 0.25) (layers F.Cu B.Cu) (net 1))
+  (via (at 139.28 113.83) (size 0.5) (drill 0.25) (layers F.Cu B.Cu) (net 1))
   (via (at 137.54 112.12) (size 0.5) (drill 0.25) (layers F.Cu B.Cu) (net 1))
   (via (at 144.91 107.78) (size 0.5) (drill 0.25) (layers F.Cu B.Cu) (net 1))
   (via (at 147.87 109.16) (size 0.5) (drill 0.25) (layers F.Cu B.Cu) (net 1))
   (via (at 142.21 108.37) (size 0.5) (drill 0.25) (layers F.Cu B.Cu) (net 1))
-  (via (at 143.72 108.9) (size 0.5) (drill 0.25) (layers F.Cu B.Cu) (net 1))
+  (via (at 143.73 108.62) (size 0.5) (drill 0.25) (layers F.Cu B.Cu) (net 1))
   (via (at 151.15 106.6) (size 0.5) (drill 0.25) (layers F.Cu B.Cu) (net 1))
   (via (at 153.46 105.28) (size 0.5) (drill 0.25) (layers F.Cu B.Cu) (net 1))
@@
   (via (at 165.01 53.47) (size 0.5) (drill 0.25) (layers F.Cu B.Cu) (net 1))
   (via (at 166.62 55.27) (size 0.5) (drill 0.25) (layers F.Cu B.Cu) (net 1))
-  (via (at 171.26 55.23) (size 0.5) (drill 0.25) (layers F.Cu B.Cu) (net 1))
+  (via (at 171.28 55.25) (size 0.5) (drill 0.25) (layers F.Cu B.Cu) (net 1))
   (via (at 171.75 56.71) (size 0.5) (drill 0.25) (layers F.Cu B.Cu) (net 1))
   (via (at 161.64 56.71) (size 0.5) (drill 0.25) (layers F.Cu B.Cu) (net 1))
@@
   (via (at 146.28 68.31) (size 0.5) (drill 0.25) (layers F.Cu B.Cu) (net 1))
   (via (at 147.08 66.64) (size 0.5) (drill 0.25) (layers F.Cu B.Cu) (net 1))
-  (via (at 149.33 65.38) (size 0.5) (drill 0.25) (layers F.Cu B.Cu) (net 1))
+  (via (at 149.41 65.4) (size 0.5) (drill 0.25) (layers F.Cu B.Cu) (net 1))
   (via (at 151.31 66.03) (size 0.5) (drill 0.25) (layers F.Cu B.Cu) (net 1))
   (via (at 153.9 66.18) (size 0.5) (drill 0.25) (layers F.Cu B.Cu) (net 1))
   (via (at 144.76 66.22) (size 0.5) (drill 0.25) (layers F.Cu B.Cu) (net 1))
   (via (at 142.67 68.66) (size 0.5) (drill 0.25) (layers F.Cu B.Cu) (net 1))
-  (via (at 143.43 73.72) (size 0.5) (drill 0.25) (layers F.Cu B.Cu) (net 1))
-  (via (at 145.71 75.93) (size 0.5) (drill 0.25) (layers F.Cu B.Cu) (net 1))
+  (via (at 143.35 73.79) (size 0.5) (drill 0.25) (layers F.Cu B.Cu) (net 1))
+  (via (at 145.58 76.05) (size 0.5) (drill 0.25) (layers F.Cu B.Cu) (net 1))
   (via (at 148.06 79.01) (size 0.5) (drill 0.25) (layers F.Cu B.Cu) (net 1))
   (via (at 152.38 79.26) (size 0.5) (drill 0.25) (layers F.Cu B.Cu) (net 1))
@@
   (via (at 141.16 75.03) (size 0.5) (drill 0.25) (layers F.Cu B.Cu) (net 1))
   (via (at 132.14 92.66) (size 0.5) (drill 0.25) (layers F.Cu B.Cu) (net 1))
-  (via (at 137.99 93.19) (size 0.5) (drill 0.25) (layers F.Cu B.Cu) (net 1))
+  (via (at 137.78 93.22) (size 0.5) (drill 0.25) (layers F.Cu B.Cu) (net 1))
   (via (at 147.79 92.86) (size 0.5) (drill 0.25) (layers F.Cu B.Cu) (net 1))
   (via (at 152.85 92.99) (size 0.5) (drill 0.25) (layers F.Cu B.Cu) (net 1))
@@
   (via (at 154.78 63.42) (size 0.5) (drill 0.25) (layers F.Cu B.Cu) (net 1))
   (via (at 151.81 63.69) (size 0.5) (drill 0.25) (layers F.Cu B.Cu) (net 1))
-  (via (at 140.28 63.66) (size 0.5) (drill 0.25) (layers F.Cu B.Cu) (net 1))
+  (via (at 140.7 63.66) (size 0.5) (drill 0.25) (layers F.Cu B.Cu) (net 1))
   (via (at 151.96 58.87) (size 0.5) (drill 0.25) (layers F.Cu B.Cu) (net 1))
   (via (at 154.63 58.33) (size 0.5) (drill 0.25) (layers F.Cu B.Cu) (net 1))
@@
   (segment (start 127.57 75.23) (end 127.54 75.26) (width 0.15) (layer F.Cu) (net 1))
   (segment (start 127.57 74.435) (end 127.57 75.23) (width 0.15) (layer F.Cu) (net 1))
-  (via (at 126.53 75.94) (size 0.5) (drill 0.25) (layers F.Cu B.Cu) (net 1))
   (via (at 127.5 76.41) (size 0.5) (drill 0.25) (layers F.Cu B.Cu) (net 1))
   (via (at 129.1 75.63) (size 0.5) (drill 0.25) (layers F.Cu B.Cu) (net 1))
+  (segment (start 128.081 71.836) (end 128.081 73.051) (width 0.15) (layer F.Cu) (net 1))
+  (segment (start 128.081 73.051) (end 128.32 73.29) (width 0.15) (layer F.Cu) (net 1))
+  (segment (start 124.76505 130.449979) (end 126.399979 130.449979) (width 0.15) (layer B.Cu) (net 1))
+  (segment (start 126.399979 130.449979) (end 126.69 130.74) (width 0.15) (layer B.Cu) (net 1))
   (segment (start 73.456 104.636) (end 73.456 107.3613) (width 0.15) (layer F.Cu) (net 2))
   (segment (start 73.456 107.3613) (end 79.8888 113.7941) (width 0.15) (layer F.Cu) (net 2))
@@
   (segment (start 112.9612 76.4743) (end 113.1265 76.309) (width 0.15) (layer F.Cu) (net 3))
   (via (at 111.9363 76.4743) (size 0.5) (layers F.Cu B.Cu) (net 3))
-  (via (at 133.09 75.04) (size 0.5) (drill 0.25) (layers F.Cu B.Cu) (net 3))
+  (via (at 133.3 75.33) (size 0.5) (drill 0.25) (layers F.Cu B.Cu) (net 3))
   (segment (start 132.3692 74.3192) (end 133.09 75.04) (width 0.15) (layer B.Cu) (net 3))
   (segment (start 131.8272 74.3192) (end 132.3692 74.3192) (width 0.15) (layer B.Cu) (net 3))
+  (segment (start 133.09 75.12) (end 133.3 75.33) (width 0.15) (layer B.Cu) (net 3))
+  (segment (start 133.09 75.04) (end 133.09 75.12) (width 0.15) (layer B.Cu) (net 3))
+  (segment (start 126.646 90.1225) (end 126.6498 90.1263) (width 0.15) (layer B.Cu) (net 3))
+  (segment (start 125.5749 90.1225) (end 126.646 90.1225) (width 0.15) (layer B.Cu) (net 3))
   (segment (start 123.406 63.161) (end 124.3187 63.161) (width 0.15) (layer F.Cu) (net 4))
   (segment (start 124.3187 63.161) (end 127.1167 65.959) (width 0.15) (layer F.Cu) (net 4))

Commit message: Generated gerber
Routing:
- net GND: track 16.8 -> 20.2 mm, vias 289 -> 291

Commit message: Generated gerber v2
Parts:
- removed C39, C40, C43, C44, C47, C48: Ccap, kifootp:CAPBUTTON
